Commit message: [nextagea_description] Further refinements to Realsense position

File: nextagea_description/urdf/NextageAOpen_gazebo_intel_realsense.urdf.xacro (robot description, xacro)
@@ -7,5 +7,5 @@
   <!-- Attach the RealSense D435 -->
   <joint name="d435_mount_joint" type="fixed">
-      <origin xyz="0 0 0.16" rpy="0 0 0"/>
+      <origin xyz="0 0 0.165" rpy="0 0.325 0"/>
       <parent link="HEAD_JOINT1_Link"/>
       <child link="d435_Mount_Link"/>

Commit message: [nextagea_description] Add inertial term to realsense mount

File: nextagea_description/urdf/NextageAOpen_gazebo_intel_realsense.urdf.xacro (robot description, xacro)
@@ -12,16 +12,9 @@
   </joint>
   <link name="d435_Mount_Link">
-    <!-- <visual>
-        <origin xyz="0 0 0" rpy="0 0 0"/>
-        <geometry>
-            <sphere radius="0.001"/>
-        </geometry>
-        <material name="DarkGrey"/>
-    </visual> -->
-    <!-- <inertial>
+    <inertial>
         <mass value="0.01"/>
         <origin rpy="0 0 0" xyz="0 0 0"/>
         <xacro:sphere_inertia_def radius="0.02" mass="0.01"/>
-    </inertial> -->
+    </inertial>
   </link>
   <xacro:sensor_d435 name="/nextagea/realsense" parent="d435_Mount_Link">
