Commit message: [nextagea_moveit_config] Topic remap fix and missing run dependency fix (#21)
* [nextagea_moveit_config] Add remap fix for MoveIt to properly read robot state

* [nextagea_moveit_config] Add missing controller manager run dependency

* [nextagea_moveit_config] Formatting fix

File: nextagea_description/urdf/NextageA_robot.xacro (robot description, xacro)
@@ -2,6 +2,6 @@
 <robot xmlns:xacro="http://ros.org/wiki/xacro">
   <xacro:include filename="$(find nextagea_description)/urdf/common.xacro" />
-  <xacro:property name="namespace" default="/nextagea/" />
-  <xacro:property name="nextagea_gazebo_ros_control" default="true" />
+  <xacro:property name="namespace" value="/nextagea/" />
+  <xacro:property name="nextagea_gazebo_ros_control" value="true" />
   <xacro:gazebo_nx_link name="WAIST" color="Black" />
   <link name="WAIST">

File: nextagea_description/urdf/common.xacro (robot description, xacro)
@@ -1,5 +1,5 @@
 <?xml version="1.0"?>
 <robot xmlns:xacro="http://ros.org/wiki/xacro">
-    <xacro:property name="nextagea_common_guard" default="true"/>
+    <xacro:property name="nextagea_common_guard" value="true"/>
     <xacro:if value="${nextagea_common_guard}">
         <xacro:property name="nextagea_common_guard" value="false"/>
