Commit message: Kinetic update to match main repo calibration

File: nextagea_description/urdf/NextageAOpen.urdf.xacro (robot description, xacro)
@@ -18,3 +18,103 @@
   <xacro:include filename="$(find nextagea_description)/urdf/NextageA_base.xacro" />
   <xacro:include filename="$(find nextagea_description)/urdf/NextageA_robot.xacro" />
+  <xacro:include filename="$(find nextagea_description)/urdf/nxao_gz_camera.xacro" />
+  <xacro:arg name="use_hand_cameras" default="false"/>
+  <xacro:arg name="use_ft_sensors" default="false"/>
+  <xacro:macro name="nxao_camera" params="prefix parent">
+    <xacro:if value="${prefix == 'L'}">
+      <xacro:property name="m" value="+1.0" />
+    </xacro:if>
+    <xacro:if value="${prefix == 'R'}">
+      <xacro:property name="m" value="-1.0" />
+    </xacro:if>
+    <xacro:gazebo_nx_link name="${prefix}ARM_camera_Link" color="Black" />
+    <link name="${prefix}ARM_camera_Link">
+      <visual>
+        <origin xyz="0 0 0" rpy="0 0 0"/>
+        <geometry>
+          <mesh filename="package://nextagea_description/urdf/meshes/${prefix}_CAM.dae"/>
+        </geometry>
+      </visual>
+      <collision>
+        <origin xyz="0 0 -0.025" rpy="0 0 0"/>
+        <geometry>
+          <cylinder length="0.05" radius="0.037"/>
+        </geometry>
+      </collision>
+      <collision>
+        <origin xyz="0.0525 ${(float(m)) * 0.029} -0.02" rpy="0 0 0"/>
+        <geometry>
+          <box size="0.057 0.106 0.042"/>
+        </geometry>
+      </collision>
+      <inertial>
+        <mass value="1.05156" />
+        <origin xyz="0.0 0.0 -0.08" rpy="0 -0 0"/>
+        <inertia ixx="0.00194072" ixy="${float(m) * 1.1e-07}" ixz="-0.00042482" iyy="0.00209392" iyz="${float(m) * 1.2e-07}" izz="0.00035788"/>
+      </inertial>
+    </link>
+    <joint name="${prefix}ARM_JOINT6" type="fixed">
+      <parent link="${parent}"/>
+      <child link="${prefix}ARM_camera_Link"/>
+      <origin xyz="0 0 0" rpy="0 0 0"/>
+      <axis xyz="0 0 1"/>
+    </joint>
+    <xacro:camera_joint_link_gzplugin
+      camera_name="CAMERA_HAND_${prefix}" link_parent="${parent}"
+      jnt_displacement_x="${jnt_hand_camera_displacement_x}"
+      jnt_displacement_y="${float(m) * jnt_hand_camera_displacement_y}"
+      jnt_displacement_z="${jnt_hand_camera_displacement_z}"
+      jnt_rotation_x="0" jnt_rotation_y="${jnt_hand_camera_rot_y}" jnt_rotation_z="0"
+      link_displacement_x="0.0325" link_displacement_y="0" link_displacement_z="0"
+      link_rotation_x="0" link_rotation_y="${M_PI/2}" link_rotation_z="-${link_hand_camera_rot_z}" />
+  </xacro:macro>
+  <xacro:macro name="nxao_ft_sensor" params="prefix parent">
+    <xacro:if value="${prefix == 'L'}">
+      <xacro:property name="m" value="+1" />
+    </xacro:if>
+    <xacro:if value="${prefix == 'R'}">
+      <xacro:property name="m" value="-1" />
+    </xacro:if>
+    <xacro:gazebo_nx_link name="${prefix}ARM_ft_Link" color="LightGrey" />
+    <link name="${prefix}ARM_ft_Link">
+      <visual>
+        <origin xyz="0 0 0.0185" rpy="0 0 0"/>
+        <geometry>
+          <cylinder length="0.037" radius="0.035"/>
+        </geometry>
+        <material name="LightGrey">
+          <color rgba="0.6 0.6 0.6 1.0"/>
+        </material>
+      </visual>
+      <collision>
+        <origin xyz="0 0 0.0185" rpy="0 0 0"/>
+        <geometry>
+          <cylinder length="0.037" radius="0.04"/>
+        </geometry>
+      </collision>
+      <!-- TODO: The inertial values are copied from ARM_JOINT5_Link. Replace with proper values. -->
+      <inertial>
+        <mass value="1.05156" />
+        <origin xyz="0.0 0.0 -0.08" rpy="0 -0 0"/>
+        <inertia ixx="0.00194072" ixy="1.1e-07" ixz="-0.00042482" iyy="0.00209392" iyz="1.2e-07" izz="0.00035788"/>
+      </inertial>
+    </link>
+    <joint name="${prefix}ARM_ft_joint" type="fixed">
+      <parent link="${parent}"/>
+      <child link="${prefix}ARM_ft_Link"/>
+      <origin xyz="0 0 -0.037" rpy="0 0 0"/>
+      <axis xyz="0 0 1"/>
+    </joint>
+  </xacro:macro>
+  <xacro:property name="arm_tip" value="ARM_JOINT5_Link" />
+  <xacro:if value="$(arg use_ft_sensors)">
+    <xacro:nxao_ft_sensor prefix="L" parent="L${arm_tip}" />
+    <xacro:nxao_ft_sensor prefix="R" parent="R${arm_tip}" />
+    <xacro:property name="arm_tip" value="ARM_ft_Link" />
+  </xacro:if>
+  <xacro:if value="$(arg use_hand_cameras)">
+    <xacro:nxao_camera prefix="L" parent="L${arm_tip}" />
+    <xacro:nxao_camera prefix="R" parent="R${arm_tip}" />
+    <xacro:property name="arm_tip" value="ARM_camera_Link" />
+  </xacro:if>
 </robot>

File: nextagea_description/urdf/NextageAOpen_gazebo_intel_realsense.urdf.xacro (robot description, xacro)
@@ -3,9 +3,137 @@
        xmlns:xacro="http://www.ros.org/wiki/xacro">
   <xacro:property name="fixed_base" value="True" />
+  <xacro:property name="ft_sensors" value="True" />
+  <xacro:property name="hand_camera" value="True" />
   <xacro:include filename="$(find nextagea_description)/urdf/NextageAOpen_gazebo.urdf.xacro" />
-  <xacro:include filename="$(find nextagea_description)/urdf/accessories/d435.urdf.xacro"/>
+  <xacro:include filename="$(find realsense2_description)/urdf/_d435.urdf.xacro"/>
+  <xacro:macro name="sensor_d435_gz" params="name">
+    <gazebo reference="${name}_color_frame">
+      <sensor name="color" type="camera">
+        <pose frame="">0 0 0 0 0 0</pose>
+        <camera name="__default__">
+          <horizontal_fov>1.5009831567151233</horizontal_fov>
+          <image>
+            <width>640</width>
+            <height>480</height>
+            <format>RGB_INT8</format>
+          </image>
+          <clip>
+            <near>0.1</near>
+            <far>100</far>
+          </clip>
+          <noise>
+            <type>gaussian</type>
+            <mean>0.0</mean>
+            <stddev>0.007</stddev>
+          </noise>
+        </camera>
+        <always_on>1</always_on>
+        <update_rate>30</update_rate>
+        <visualize>1</visualize>
+      </sensor>
+    </gazebo>
+    <gazebo reference="${name}_infra1_frame">
+      <sensor name="ired1" type="camera">
+        <pose frame="">0 0 0 0 0 0</pose>
+        <camera name="__default__">
+          <horizontal_fov>1.5009831567151233</horizontal_fov>
+          <image>
+            <width>640</width>
+            <height>480</height>
+            <format>L_INT8</format>
+          </image>
+          <clip>
+            <near>0.1</near>
+            <far>100</far>
+          </clip>
+          <noise>
+            <type>gaussian</type>
+            <mean>0.0</mean>
+            <stddev>0.007</stddev>
+          </noise>
+        </camera>
+        <always_on>1</always_on>
+        <update_rate>30</update_rate>
+        <visualize>0</visualize>
+      </sensor>
+    </gazebo>
+    <gazebo reference="${name}_infra2_frame">
+      <sensor name="ired2" type="camera">
+        <pose frame="">0 0 0 0 0 0</pose>
+        <camera name="__default__">
+          <horizontal_fov>1.5009831567151233</horizontal_fov>
+          <image>
+            <width>640</width>
+            <height>480</height>
+            <format>L_INT8</format>
+          </image>
+          <clip>
+            <near>0.1</near>
+            <far>100</far>
+          </clip>
+          <noise>
+            <type>gaussian</type>
+            <mean>0.0</mean>
+            <stddev>0.007</stddev>
+          </noise>
+        </camera>
+        <always_on>1</always_on>
+        <update_rate>30</update_rate>
+        <visualize>0</visualize>
+      </sensor>
+    </gazebo>
+    <gazebo reference="${name}_depth_frame">
+      <sensor name="depth" type="depth">
+        <pose frame="">0 0 0 0 0 0</pose>
+        <camera name="__default__">
+          <horizontal_fov>1.5009831567151233</horizontal_fov>
+          <image>
+            <width>640</width>
+            <height>480</height>
+          </image>
+          <clip>
+            <near>0.1</near>
+            <far>100</far>
+          </clip>
+          <noise>
+            <type>gaussian</type>
+            <mean>0.0</mean>
+            <stddev>0.007</stddev>
+          </noise>
+        </camera>
+        <always_on>1</always_on>
+        <update_rate>30</update_rate>
+        <visualize>0</visualize>
+      </sensor>
+    </gazebo>
+    <gazebo>
+      <plugin name="${name}" filename="librealsense_gazebo_plugin.so">
+        <depthUpdateRate>30</depthUpdateRate>
+        <colorUpdateRate>30</colorUpdateRate>
+        <infraredUpdateRate>30</infraredUpdateRate>
+        <depthTopicName>depth/image_raw</depthTopicName>
+        <depthCameraInfoTopicName>depth/camera_info</depthCameraInfoTopicName>
+        <colorTopicName>color/image_raw</colorTopicName>
+        <colorCameraInfoTopicName>color/camera_info</colorCameraInfoTopicName>
+        <infrared1TopicName>infrared/image_raw</infrared1TopicName>
+        <infrared1CameraInfoTopicName>infrared/camera_info</infrared1CameraInfoTopicName>
+        <infrared2TopicName>infrared2/image_raw</infrared2TopicName>
+        <infrared2CameraInfoTopicName>infrared2/camera_info</infrared2CameraInfoTopicName>
+        <colorOpticalframeName>camera_color_optical_frame</colorOpticalframeName>
+        <depthOpticalframeName>camera_depth_optical_frame</depthOpticalframeName>
+        <infrared1OpticalframeName>camera_left_ir_optical_frame</infrared1OpticalframeName>
+        <infrared2OpticalframeName>camera_right_ir_optical_frame</infrared2OpticalframeName>
+        <rangeMinDepth>0.1</rangeMinDepth>
+        <rangeMaxDepth>10</rangeMaxDepth>
+        <pointCloud>1</pointCloud>
+        <pointCloudTopicName>depth/color/points</pointCloudTopicName>
+        <pointCloudCutoff>0.15</pointCloudCutoff>
+        <pointCloudCutoffMax>10</pointCloudCutoffMax>
+      </plugin>
+    </gazebo>
+  </xacro:macro>
   <!-- Attach the RealSense D435 -->
   <joint name="d435_mount_joint" type="fixed">
-      <origin xyz="0 0 0.165" rpy="0 0.325 0"/>
+      <origin xyz="0 0 0.1448322" rpy="0 0.24902114520034205 0"/>
       <parent link="HEAD_JOINT1_Link"/>
       <child link="d435_Mount_Link"/>
@@ -18,6 +146,7 @@
     </inertial>
   </link>
-  <xacro:sensor_d435 name="/nextagea/realsense" parent="d435_Mount_Link">
+  <xacro:sensor_d435 name="nextagea_realsense" parent="d435_Mount_Link" use_nominal_extrinsics="true">
       <origin xyz="0 0 0" rpy="0 0 0"/>
   </xacro:sensor_d435>
+  <xacro:sensor_d435_gz name="nextagea_realsense" />
 </robot>

File: nextagea_description/urdf/NextageA_robot.xacro (robot description, xacro)
@@ -2,6 +2,8 @@
 <robot xmlns:xacro="http://www.ros.org/wiki/xacro">
   <xacro:include filename="$(find nextagea_description)/urdf/common.xacro" />
-  <xacro:property name="namespace" value="/nextagea/" />
-  <xacro:property name="nextagea_gazebo_ros_control" value="true" />
+  <xacro:arg name="namespace_arg" default="/nextagea/"/>
+  <xacro:arg name="nextagea_gazebo_ros_control_arg" default="true"/>
+  <xacro:property name="namespace" value="$(arg namespace_arg)" />
+  <xacro:property name="nextagea_gazebo_ros_control" value="$(arg nextagea_gazebo_ros_control_arg)" />
   <xacro:gazebo_nx_link name="WAIST" color="Black" />
   <link name="WAIST">
@@ -276,20 +278,8 @@
       </geometry>
     </visual>
-    <visual>
-      <origin xyz="0 0 0" rpy="0 0 0"/>
-      <geometry>
-	      <mesh filename="package://nextagea_description/urdf/meshes/L_CAM.dae"/>
-      </geometry>
-    </visual>
-    <collision>
-      <origin xyz="0 0 -0.02" rpy="0 0 0"/>
-      <geometry>
-        <cylinder length="0.07" radius="0.037"/>
-      </geometry>
-    </collision>
-    <collision>
-      <origin xyz="0.0525 0.029 -0.02" rpy="0 0 0"/>
-      <geometry>
-        <box size="0.057 0.106 0.042"/>
+    <collision>
+      <origin xyz="0 0 0.0065" rpy="0 0 0"/>
+      <geometry>
+        <cylinder length="0.013" radius="0.037"/>
       </geometry>
     </collision>
@@ -456,20 +446,8 @@
       </geometry>
     </visual>
-    <visual>
-      <origin xyz="0 0 0" rpy="0 0 0"/>
-      <geometry>
-	      <mesh filename="package://nextagea_description/urdf/meshes/R_CAM.dae"/>
-      </geometry>
-    </visual>
-    <collision>
-      <origin xyz="0 0 -0.02" rpy="0 0 0"/>
-      <geometry>
-        <cylinder length="0.07" radius="0.037"/>
-      </geometry>
-    </collision>
-    <collision>
-      <origin xyz="0.0525 -0.029 -0.02" rpy="0 0 0"/>
-      <geometry>
-        <box size="0.057 0.106 0.042"/>
+    <collision>
+      <origin xyz="0 0 0.0065" rpy="0 0 0"/>
+      <geometry>
+        <cylinder length="0.013" radius="0.037"/>
       </geometry>
     </collision>
@@ -618,5 +596,5 @@
       <plugin name="gazebo_ros_control" filename="libgazebo_ros_control.so">
         <robotNamespace>${namespace}</robotNamespace>
-        <legacyModeNS>true</legacyModeNS>
+         <legacyModeNS>true</legacyModeNS>
       </plugin>
     </gazebo>

File: nextagea_description/urdf/common.xacro (robot description, xacro)
@@ -1,5 +1,6 @@
 <?xml version="1.0"?>
 <robot xmlns:xacro="http://www.ros.org/wiki/xacro">
-    <xacro:property name="nextagea_common_guard" value="true"/>
+    <xacro:arg name="nextagea_common_guard_flag" default="true"/>
+    <xacro:property name="nextagea_common_guard" value="$(arg nextagea_common_guard_flag)"/>
     <xacro:if value="${nextagea_common_guard}">
         <xacro:property name="nextagea_common_guard" value="false"/>
@@ -18,8 +19,8 @@
             <type>transmission_interface/SimpleTransmission</type>
             <joint name="${name}">
-                <hardwareInterface>hardware_interface/PositionJointInterface</hardwareInterface>/hardwareInterface>
+                <hardwareInterface>hardware_interface/PositionJointInterface</hardwareInterface>
             </joint>
             <actuator name="${name}_Motor">
-                <hardwareInterface>hardware_interface/PositionJointInterface</hardwareInterface>/hardwareInterface>
+                <hardwareInterface>hardware_interface/PositionJointInterface</hardwareInterface>
                 <mechanicalReduction>1</mechanicalReduction>
             </actuator>
